File: kicad project/micropsu.kicad_pcb (KiCad board)
At the start: 2 copper layers, 62 x 78 mm, 17 parts, among them P78E12-1000 VXO7805-1000, Q1 FQP47P06, SW1 SS-22G88-G090, U1 B2P-VH-BL(LF)(SN), U3 dfr0831V2

Commit message: updated version of board
Parts:
- added +12V ALT Input: BarrelJack_Kycon_KLDX-0202-xC_Horizontal, Connector_BarrelJack:BarrelJack_Kycon_KLDX-0202-xC_Horizontal, F.Cu at (115.7, 90.2)
- SW1: value SS-22G88-G090 -> 500SDP1S1M2QEA; footprint SW-TH_G-SWITC_SS-22G88-G090 -> footprints:SW6_M2QEA_EWI
- moved SW1 6.24 mm to (95.5, 93.3), turned to 90 degrees
- moved +5INPUT 5.50 mm to (125.5, 104.0), turned to -90 degrees
- moved -5INPUT 4.89 mm to (116.5, 97.0), turned to 0 degrees
- moved LED1 2.60 mm to (146.5, 141.0)
- renumbered U1 to J1, Output to J2
Connections:
- SW1 pad 1: (no net) -> +12V
- SW1 pad 3: +12V -> (no net)
- SW1 pad 4: +12V -> (no net)
- SW1 pad 6: (no net) -> +12V
Routing:
- net +12V: track 214.3 -> 215.0 mm
Other:
- board text added: "* CHECK VOLTAGE PINOUT ON"
- board text added: "* WARNING: USE J1 or J3 - NOT BOTH!"
- board text added: "+tip"
- board text added: "09652028"
- board text added: "26604040"
- board text added: "J3"
- board text added: "ORIGINAL BOARD!"
- board text added: "Output"
- board text added: "SW1"
- board text added: "WE 694106301002"
- board text added: "hexbus MSX microPSU +-12V/5V 1.0c 10/2024"
- board text removed: "CHECK VOLTAGE PINOUT"
- board text removed: "ON ORIGINAL BOARD"
- board text removed: "hexbus MSX microPSU +-12V/5V 1.0b 10/2024"
